File: hardware/megadrive_adapter/megadrive_adapter.kicad_pcb (KiCad board)
At the start: 2 copper layers, 96.6 x 25.5 mm, 3 parts, among them J1 CART SLOT TOP ROW, J2 CART SLOT BOTTOM ROW, U1 MD_Slot

Commit message: megadrive adapter: update main label; -> kicad v7
Other:
- board text added: "M E G A D R I V E"
- board text removed: "2.54mm 64-Pin MEGA DRIVE Cartridge Slot"
